File: Highside-powerdistribution/Highside-powerdistribution.sch (KiCad schematic (older format))
At the start: 43 parts, among them J1 Conn_01x02_Male, J10 Screw_Terminal_01x02, J11 Screw_Terminal_01x02, J12 Screw_Terminal_01x02, J13 Screw_Terminal_01x02, J14 Conn_01x02, J15 Screw_Terminal_01x06, J2 Conn_01x02_Male, J3 Conn_01x02_Male, J4 Conn_01x02_Male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

Commit message: Changed to terminal block on input
Parts:
- J14: footprint Highside-powerdistribution:XT60PW-F -> Highside-powerdistribution:Phoenix_TB_2-1935776
Changed lines of the file:
@@
 F 0 "J14" H 9130 3192 50  0000 L CNN
 F 1 "Conn_01x02" H 9130 3101 50  0000 L CNN
-F 2 "Highside-powerdistribution:XT60PW-F" H 9050 3200 50  0001 C CNN
+F 2 "Highside-powerdistribution:Phoenix_TB_2-1935776" H 9050 3200 50  0001 C CNN
 F 3 "~" H 9050 3200 50  0001 C CNN
 	1    9050 3200
