File: hardware/power-distribution/power-distribution.kicad_pcb (KiCad board)
At the start: 2 copper layers, 90 x 70 mm, 25 parts, among them J1 Parallell, J2 Parallell, J3 Parallell, Q1 Q_PMOS_GDS, Q2 Q_PMOS_GDS, Q3 Q_PMOS_GDS, Q4 Q_PMOS_GDS

Commit message: Changed to 7.62 input pitch and 8 output with 2 and 2
Parts:
- removed POWER_OUT1: Screw_Terminal_01x04, TerminalBlock_Phoenix:TerminalBlock_Phoenix_PT-1,5-4-5.0-H_1x04_P5.00mm_Horizontal
- added J4: Screw_Terminal_01x08, TerminalBlock_Phoenix:TerminalBlock_Phoenix_MKDS-1,5-8_1x08_P5.00mm_Horizontal, F.Cu at (120.0, 125.0)
- POWER_IN1: footprint TerminalBlock_Phoenix:TerminalBlock_Phoenix_PT-1,5-2-5.0-H_1x02_P5.00mm_Horizontal -> TerminalBlock:TerminalBlock_Wuerth_691311400102_P7.62mm
