File: hardware/led-dimmer/led_dimmer.sch (KiCad schematic (older format))
At the start: 5 parts

Commit message: Added terminal block, LDO and connected mosfet
Parts:
- removed J?: Screw_Terminal_01x02, symbol Connector:Screw_Terminal_01x02
- added C? (x3): C, symbol Device:C
- added J?: Screw_Terminal_01x03, symbol Connector:Screw_Terminal_01x03
- added R?: 1k, symbol Device:R
Connections:
- net labels added: +12V, +3V3, +VSW, GND, LED_DIMMER
- wire segments 0 -> 21
Other:
- moved on the sheet: U?

Commit message: Added power OR-circuit for 5V and 12V
Parts:
- removed C? (x3): C, symbol Device:C
- removed R?: 1k, symbol Device:R
- added C1, C2, C3, C4, C5, C6: C_Small, Capacitor_SMD:C_0603_1608Metric, symbol Device:C_Small
- added D1, D2: D_Small, Diode_SMD:D_SOD-123, symbol Device:D_Small
- added J1: USB_B_Micro, symbol Connector:USB_B_Micro
- added R1, R2: 10k, Resistor_SMD:R_0603_1608Metric, symbol Device:R_Small
- added R3, R6: 1k, Resistor_SMD:R_0603_1608Metric, symbol Device:R_Small
- added R4: 100k, Resistor_SMD:R_0603_1608Metric, symbol Device:R_Small
- added R5: R_Small, Resistor_SMD:R_0603_1608Metric, symbol Device:R_Small
- added SW2: ~Reset, symbol Switch:SW_Push
- added SWD1: SWD_TAGCONNECT, symbol connector:SWD_TAGCONNECT
- gave numbers to parts that had none: 5
Connections:
- net labels added: +5V, A1, A2, A3, A4, D0, D1, D10, D11_ENCB, D13_ENC_SW, D2, D3_LED, D4, D5_ENCA, D8, D9, SCL, SDA, SWCLK, SWDIO, USB+, USB-, ~RESET
- net labels removed: LED_DIMMER
- wire segments 21 -> 70
- no-connect marks 0 -> 1
Other:
- note added: "12V if possible, otherwise 5V"
- moved on the sheet: SW1

Commit message: Added two mosfets for pull both to GND.
Parts:
- removed J2: Screw_Terminal_01x03, symbol Connector:Screw_Terminal_01x03
- removed Q1: Q_NMOS_DGS, symbol Device:Q_NMOS_DGS
- added J2: Screw_Terminal_01x04, symbol Connector:Screw_Terminal_01x04
- added Q1, Q2: Q_NMOS_GSD, Package_TO_SOT_SMD:SOT-23, symbol Device:Q_NMOS_GSD
- added R7: 1k, Resistor_SMD:R_0603_1608Metric, symbol Device:R_Small
- J1: footprint (none) -> connectors:Microusb_105133-0011
- SW1: footprint (none) -> Rotary_Encoder:RotaryEncoder_Alps_EC11E-Switch_Vertical_H20mm
- SWD1: footprint (none) -> connectors:TAG_TC2030-IDC-NL
Connections:
- net labels added: SWA, SWB
- net labels removed: +VSW
- wire segments 70 -> 74
Changed lines of the file:
@@
 F 0 "SW1" H 2050 3017 50  0000 C CNN
 F 1 "Rotary_Encoder_Switch" H 2050 2926 50  0000 C CNN
-F 2 "" H 1900 2810 50  0001 C CNN
+F 2 "Rotary_Encoder:RotaryEncoder_Alps_EC11E-Switch_Vertical_H20mm" H 1900 2810 50  0001 C CNN
 F 3 "~" H 2050 2910 50  0001 C CNN
 	1    2050 2650
-	1    0    0    -1
-$EndComp
-$Comp
-L Device:Q_NMOS_DGS Q1
-U 1 1 5E87677D
-P 8450 2550
-F 0 "Q1" H 8656 2596 50  0000 L CNN
-F 1 "Q_NMOS_DGS" H 8656 2505 50  0000 L CNN
-F 2 "" H 8650 2650 50  0001 C CNN
-F 3 "~" H 8450 2550 50  0001 C CNN
-	1    8450 2550
 	1    0    0    -1
 $EndComp
@@
 $EndComp
 $Comp
-L Connector:Screw_Terminal_01x03 J2
-U 1 1 5E8852F4
-P 8300 3900
-F 0 "J2" H 8380 3942 50  0000 L CNN
-F 1 "Screw_Terminal_01x03" H 8380 3851 50  0000 L CNN
-F 2 "" H 8300 3900 50  0001 C CNN
-F 3 "~" H 8300 3900 50  0001 C CNN
-	1    8300 3900
-	1    0    0    -1
-$EndComp
-$Comp
 L power:+12V #PWR0101
 U 1 1 5E885A1F
@@
 L power:GND #PWR0102
 U 1 1 5E886277
-P 8000 4100
-F 0 "#PWR0102" H 8000 3850 50  0001 C CNN
-F 1 "GND" H 8005 3927 50  0000 C CNN
-F 2 "" H 8000 4100 50  0001 C CNN
-F 3 "" H 8000 4100 50  0001 C CNN
-	1    8000 4100
-	1    0    0    -1
-$EndComp
-$Comp
-L power:+VSW #PWR0103
-U 1 1 5E886D33
-P 7800 3700
-F 0 "#PWR0103" H 7800 3550 50  0001 C CNN
-F 1 "+VSW" H 7815 3873 50  0000 C CNN
-F 2 "" H 7800 3700 50  0001 C CNN
-F 3 "" H 7800 3700 50  0001 C CNN
-	1    7800 3700
-	1    0    0    -1
-$EndComp
-Wire Wire Line
-	7800 3700 7800 3900
-Wire Wire Line
-	7800 3900 8100 3900
+P 8000 4000
+F 0 "#PWR0102" H 8000 3750 50  0001 C CNN
+F 1 "GND" H 8005 3827 50  0000 C CNN
+F 2 "" H 8000 4000 50  0001 C CNN
+F 3 "" H 8000 4000 50  0001 C CNN
+	1    8000 4000
+	1    0    0    -1
+$EndComp
 Wire Wire Line
 	8000 3700 8000 3800
 Wire Wire Line
-	8000 3800 8100 3800
-Wire Wire Line
-	8100 4000 8000 4000
-Wire Wire Line
-	8000 4000 8000 4100
+	8000 3900 8000 4000
 $Comp
 L power:GND #PWR0104
@@
 F 3 "" H 8150 2950 50  0001 C CNN
 	1    8150 2950
-	1    0    0    -1
-$EndComp
-$Comp
-L power:+VSW #PWR0105
-U 1 1 5E88D369
-P 8550 2250
-F 0 "#PWR0105" H 8550 2100 50  0001 C CNN
-F 1 "+VSW" H 8565 2423 50  0000 C CNN
-F 2 "" H 8550 2250 50  0001 C CNN
-F 3 "" H 8550 2250 50  0001 C CNN
-	1    8550 2250
 	1    0    0    -1
 $EndComp
@@
 F 0 "J1" H 1707 4317 50  0000 C CNN
 F 1 "USB_B_Micro" H 1707 4226 50  0000 C CNN
-F 2 "" H 1800 3800 50  0001 C CNN
+F 2 "connectors:Microusb_105133-0011" H 1800 3800 50  0001 C CNN
 F 3 "~" H 1800 3800 50  0001 C CNN
 	1    1650 3850
@@
 F 0 "SWD1" H 2500 1870 50  0000 C CNN
 F 1 "SWD_TAGCONNECT" H 2500 1779 50  0000 C CNN
-F 2 "" H 2500 1500 50  0001 C CNN
+F 2 "connectors:TAG_TC2030-IDC-NL" H 2500 1500 50  0001 C CNN
 F 3 "" H 2500 1500 50  0001 C CNN
 	1    2500 1500
@@
 Text Notes 6700 4450 0    50   ~ 0
 12V if possible, otherwise 5V
+$Comp
+L power:GND #PWR0103
+U 1 1 5E895722
+P 9700 2950
+F 0 "#PWR0103" H 9700 2700 50  0001 C CNN
+F 1 "GND" H 9705 2777 50  0000 C CNN
+F 2 "" H 9700 2950 50  0001 C CNN
+F 3 "" H 9700 2950 50  0001 C CNN
+	1    9700 2950
+	1    0    0    -1
+$EndComp
+$Comp
+L power:GND #PWR0105
+U 1 1 5E89572E
+P 10100 2850
+F 0 "#PWR0105" H 10100 2600 50  0001 C CNN
+F 1 "GND" H 10105 2677 50  0000 C CNN
+F 2 "" H 10100 2850 50  0001 C CNN
+F 3 "" H 10100 2850 50  0001 C CNN
+	1    10100 2850
+	1    0    0    -1
+$EndComp
+Wire Wire Line
+	10100 2850 10100 2750
+Wire Wire Line
+	10100 2350 10100 2250
+Wire Wire Line
+	9800 2550 9700 2550
+Wire Wire Line
+	9700 2550 9700 2650
+Wire Wire Line
+	9700 2850 9700 2950
+Wire Wire Line
+	9700 2550 9600 2550
+Connection ~ 9700 2550
+$Comp
+L Device:R_Small R7
+U 1 1 5E89573B
+P 9700 2750
+F 0 "R7" H 9759 2796 50  0000 L CNN
+F 1 "1k" H 9759 2705 50  0000 L CNN
+F 2 "Resistor_SMD:R_0603_1608Metric" H 9700 2750 50  0001 C CNN
+F 3 "~" H 9700 2750 50  0001 C CNN
+	1    9700 2750
+	1    0    0    -1
+$EndComp
+Text GLabel 9600 2550 0    50   Input ~ 0
+D3_LED
+$Comp
+L Connector:Screw_Terminal_01x04 J2
+U 1 1 5E89857B
+P 8450 3900
+F 0 "J2" H 8530 3892 50  0000 L CNN
+F 1 "Screw_Terminal_01x04" H 8530 3801 50  0000 L CNN
+F 2 "" H 8450 3900 50  0001 C CNN
+F 3 "~" H 8450 3900 50  0001 C CNN
+	1    8450 3900
+	1    0    0    -1
+$EndComp
+Wire Wire Line
+	8000 3900 8250 3900
+Wire Wire Line
+	8000 3800 8250 3800
+Text GLabel 8250 4000 0    50   Input ~ 0
+SWA
+Text GLabel 8250 4100 0    50   Input ~ 0
+SWB
+Text GLabel 8550 2250 0    50   Input ~ 0
+SWA
+Text GLabel 10100 2250 0    50   Input ~ 0
+SWB
+$Comp
+L Device:Q_NMOS_GSD Q2
+U 1 1 5E8A6696
+P 10000 2550
+F 0 "Q2" H 10206 2596 50  0000 L CNN
+F 1 "Q_NMOS_GSD" H 10206 2505 50  0000 L CNN
+F 2 "Package_TO_SOT_SMD:SOT-23" H 10200 2650 50  0001 C CNN
+F 3 "~" H 10000 2550 50  0001 C CNN
+	1    10000 2550
+	1    0    0    -1
+$EndComp
+$Comp
+L Device:Q_NMOS_GSD Q1
+U 1 1 5E8A804C
+P 8450 2550
+F 0 "Q1" H 8656 2596 50  0000 L CNN
+F 1 "Q_NMOS_GSD" H 8656 2505 50  0000 L CNN
+F 2 "Package_TO_SOT_SMD:SOT-23" H 8650 2650 50  0001 C CNN
+F 3 "~" H 8450 2550 50  0001 C CNN
+	1    8450 2550
+	1    0    0    -1
+$EndComp
 $EndSCHEMATC

Commit message: Removed "unnecessary" components
Parts:
- removed C2: C_Small, Capacitor_SMD:C_0603_1608Metric, symbol Device:C_Small
- removed R7: 1k, Resistor_SMD:R_0603_1608Metric, symbol Device:R_Small
- removed SW2: ~Reset, symbol Switch:SW_Push
- added Q3, Q4: Q_PMOS_GDS, symbol Device:Q_PMOS_GDS
- J2: footprint (none) -> TerminalBlock_Phoenix:TerminalBlock_Phoenix_MKDS-3-4-5.08_1x04_P5.08mm_Horizontal
- R5: value R_Small -> Dummy; footprint Resistor_SMD:R_0603_1608Metric -> Resistor_SMD:R_0402_1005Metric
Connections:
- net labels added: D4_PMOS_SWA, D9_PMOS_SWA
- net labels removed: D4, D9
- wire segments 74 -> 71
Changed lines of the file:
@@
 Connection ~ 8700 5000
 Connection ~ 7700 5000
-Wire Wire Line
-	3650 5000 3750 5000
-$Comp
-L power:GND #PWR0112
-U 1 1 5E873923
-P 3750 5400
-F 0 "#PWR0112" H 3750 5150 50  0001 C CNN
-F 1 "GND" H 3755 5227 50  0000 C CNN
-F 2 "" H 3750 5400 50  0001 C CNN
-F 3 "" H 3750 5400 50  0001 C CNN
-	1    3750 5400
-	1    0    0    -1
-$EndComp
-Wire Wire Line
-	3750 5400 3750 5300
-Wire Wire Line
-	3750 5100 3750 5000
-Connection ~ 3750 5000
-Wire Wire Line
-	3750 5000 4100 5000
-$Comp
-L Device:C_Small C2
-U 1 1 5E874927
-P 3750 5200
-F 0 "C2" H 3842 5246 50  0000 L CNN
-F 1 "C_Small" H 3842 5155 50  0000 L CNN
-F 2 "Capacitor_SMD:C_0603_1608Metric" H 3750 5200 50  0001 C CNN
-F 3 "~" H 3750 5200 50  0001 C CNN
-	1    3750 5200
-	1    0    0    -1
-$EndComp
 $Comp
 L Device:C_Small C6
@@
 L power:GND #PWR0113
 U 1 1 5E8781D5
-P 2850 5100
-F 0 "#PWR0113" H 2850 4850 50  0001 C CNN
-F 1 "GND" H 2855 4927 50  0000 C CNN
-F 2 "" H 2850 5100 50  0001 C CNN
-F 3 "" H 2850 5100 50  0001 C CNN
-	1    2850 5100
-	1    0    0    -1
-$EndComp
-$Comp
-L Switch:SW_Push SW2
-U 1 1 5E87A145
-P 3150 5000
-F 0 "SW2" H 3150 5297 50  0000 C CNN
-F 1 "~Reset" H 3150 5199 50  0000 C CNN
-F 2 "" H 3150 5200 50  0001 C CNN
-F 3 "~" H 3150 5200 50  0001 C CNN
-	1    3150 5000
-	1    0    0    -1
-$EndComp
-Wire Wire Line
-	2850 5100 2850 5000
-Wire Wire Line
-	2850 5000 2950 5000
+P 3250 5100
+F 0 "#PWR0113" H 3250 4850 50  0001 C CNN
+F 1 "GND" H 3255 4927 50  0000 C CNN
+F 2 "" H 3250 5100 50  0001 C CNN
+F 3 "" H 3250 5100 50  0001 C CNN
+	1    3250 5100
+	1    0    0    -1
+$EndComp
+Wire Wire Line
+	3250 5100 3250 5000
 $Comp
 L Device:R_Small R6
@@
 P 3550 5000
 F 0 "R5" V 3746 5000 50  0000 C CNN
-F 1 "R_Small" V 3655 5000 50  0000 C CNN
-F 2 "Resistor_SMD:R_0603_1608Metric" H 3550 5000 50  0001 C CNN
+F 1 "Dummy" V 3655 5000 50  0000 C CNN
+F 2 "Resistor_SMD:R_0402_1005Metric" H 3550 5000 50  0001 C CNN
 F 3 "~" H 3550 5000 50  0001 C CNN
 	1    3550 5000
 	0    -1   -1   0
 $EndComp
-Wire Wire Line
-	3450 5000 3350 5000
 $Comp
 L power:GND #PWR0114
@@
 Text GLabel 4100 2500 0    50   Input ~ 0
 D8
-Text GLabel 4100 2600 0    50   Input ~ 0
-D9
-Text GLabel 4100 2700 0    50   Input ~ 0
-D4
 Text GLabel 4100 2800 0    50   Input ~ 0
 D3_LED
@@
 12V if possible, otherwise 5V
 $Comp
-L power:GND #PWR0103
-U 1 1 5E895722
-P 9700 2950
-F 0 "#PWR0103" H 9700 2700 50  0001 C CNN
-F 1 "GND" H 9705 2777 50  0000 C CNN
-F 2 "" H 9700 2950 50  0001 C CNN
-F 3 "" H 9700 2950 50  0001 C CNN
-	1    9700 2950
-	1    0    0    -1
-$EndComp
-$Comp
 L power:GND #PWR0105
 U 1 1 5E89572E
@@
 Wire Wire Line
 	10100 2350 10100 2250
-Wire Wire Line
-	9800 2550 9700 2550
-Wire Wire Line
-	9700 2550 9700 2650
-Wire Wire Line
-	9700 2850 9700 2950
-Wire Wire Line
-	9700 2550 9600 2550
-Connection ~ 9700 2550
-$Comp
-L Device:R_Small R7
-U 1 1 5E89573B
-P 9700 2750
-F 0 "R7" H 9759 2796 50  0000 L CNN
-F 1 "1k" H 9759 2705 50  0000 L CNN
-F 2 "Resistor_SMD:R_0603_1608Metric" H 9700 2750 50  0001 C CNN
-F 3 "~" H 9700 2750 50  0001 C CNN
-	1    9700 2750
-	1    0    0    -1
-$EndComp
 Text GLabel 9600 2550 0    50   Input ~ 0
 D3_LED
@@
 F 0 "J2" H 8530 3892 50  0000 L CNN
 F 1 "Screw_Terminal_01x04" H 8530 3801 50  0000 L CNN
-F 2 "" H 8450 3900 50  0001 C CNN
+F 2 "TerminalBlock_Phoenix:TerminalBlock_Phoenix_MKDS-3-4-5.08_1x04_P5.08mm_Horizontal" H 8450 3900 50  0001 C CNN
 F 3 "~" H 8450 3900 50  0001 C CNN
 	1    8450 3900
@@
 	1    0    0    -1
 $EndComp
+$Comp
+L power:+12V #PWR0130
+U 1 1 5E890108
+P 8500 1250
+F 0 "#PWR0130" H 8500 1100 50  0001 C CNN
+F 1 "+12V" H 8515 1423 50  0000 C CNN
+F 2 "" H 8500 1250 50  0001 C CNN
+F 3 "" H 8500 1250 50  0001 C CNN
+	1    8500 1250
+	1    0    0    -1
+$EndComp
+$Comp
+L Device:Q_PMOS_GDS Q3
+U 1 1 5E88F1EF
+P 8400 1500
+F 0 "Q3" H 8606 1454 50  0000 L CNN
+F 1 "Q_PMOS_GDS" H 8606 1545 50  0000 L CNN
+F 2 "" H 8600 1600 50  0001 C CNN
+F 3 "~" H 8400 1500 50  0001 C CNN
+	1    8400 1500
+	1    0    0    1
+$EndComp
+Wire Wire Line
+	8500 1250 8500 1300
+Wire Wire Line
+	8500 1700 8500 1750
+Text GLabel 8500 1750 0    50   Input ~ 0
+SWA
+$Comp
+L Device:Q_PMOS_GDS Q4
+U 1 1 5E89A113
+P 9850 1500
+F 0 "Q4" H 10056 1454 50  0000 L CNN
+F 1 "Q_PMOS_GDS" H 10056 1545 50  0000 L CNN
+F 2 "" H 10050 1600 50  0001 C CNN
+F 3 "~" H 9850 1500 50  0001 C CNN
+	1    9850 1500
+	1    0    0    1
+$EndComp
+Text GLabel 9950 1750 0    50   Input ~ 0
+SWB
+Wire Wire Line
+	9950 1700 9950 1750
+$Comp
+L power:+12V #PWR0131
+U 1 1 5E89CF4D
+P 9950 1250
+F 0 "#PWR0131" H 9950 1100 50  0001 C CNN
+F 1 "+12V" H 9965 1423 50  0000 C CNN
+F 2 "" H 9950 1250 50  0001 C CNN
+F 3 "" H 9950 1250 50  0001 C CNN
+	1    9950 1250
+	1    0    0    -1
+$EndComp
+Wire Wire Line
+	9950 1250 9950 1300
+Text GLabel 8150 1500 0    50   Input ~ 0
+D4_PMOS_SWA
+Text GLabel 9600 1500 0    50   Input ~ 0
+D9_PMOS_SWA
+Text GLabel 4100 2700 0    50   Input ~ 0
+D4_PMOS_SWA
+Text GLabel 4100 2600 0    50   Input ~ 0
+D9_PMOS_SWA
+Wire Wire Line
+	9600 2550 9800 2550
+Wire Wire Line
+	3650 5000 4100 5000
+Wire Wire Line
+	3250 5000 3450 5000
 $EndSCHEMATC

Commit message: Changed to just Pmosfet
Parts:
- removed J2: Screw_Terminal_01x04, TerminalBlock_Phoenix:TerminalBlock_Phoenix_MKDS-3-4-5.08_1x04_P5.08mm_Horizontal, symbol Connector:Screw_Terminal_01x04
- removed Q1, Q2: Q_NMOS_GSD, Package_TO_SOT_SMD:SOT-23, symbol Device:Q_NMOS_GSD
- removed Q3: Q_PMOS_GDS, symbol Device:Q_PMOS_GDS
- removed R6: 1k, Resistor_SMD:R_0603_1608Metric, symbol Device:R_Small
- added F1: Fuse_Small, Private Fuses:ATO_Fuseholder_3522-2, symbol Device:Fuse_Small
- added J2: Screw_Terminal_01x03, TerminalBlock_Phoenix:TerminalBlock_Phoenix_MKDS-1,5-3_1x03_P5.00mm_Horizontal, symbol Connector:Screw_Terminal_01x03
- added Q3: Q_NMOS_GSD, Package_TO_SOT_SMD:SOT-23, symbol Device:Q_NMOS_GSD
- added R7, R8: 1k, Resistor_SMD:R_0603_1608Metric, symbol Device:R_Small
- Q4: footprint (none) -> Package_TO_SOT_SMD:TO-252-2
Connections:
- net labels added: D8_LED_POWER, LED
- net labels removed: D8, SWA, SWB
- wire segments 71 -> 69
Changed lines of the file:
@@
 L power:+12V #PWR0101
 U 1 1 5E885A1F
-P 8000 3700
-F 0 "#PWR0101" H 8000 3550 50  0001 C CNN
-F 1 "+12V" H 8015 3873 50  0000 C CNN
-F 2 "" H 8000 3700 50  0001 C CNN
-F 3 "" H 8000 3700 50  0001 C CNN
-	1    8000 3700
+P 7850 3700
+F 0 "#PWR0101" H 7850 3550 50  0001 C CNN
+F 1 "+12V" H 7865 3873 50  0000 C CNN
+F 2 "" H 7850 3700 50  0001 C CNN
+F 3 "" H 7850 3700 50  0001 C CNN
+	1    7850 3700
 	1    0    0    -1
 $EndComp
@@
 $EndComp
 Wire Wire Line
-	8000 3700 8000 3800
+	7850 3700 7850 3800
 Wire Wire Line
 	8000 3900 8000 4000
-$Comp
-L power:GND #PWR0104
-U 1 1 5E88CCFB
-P 8150 2950
-F 0 "#PWR0104" H 8150 2700 50  0001 C CNN
-F 1 "GND" H 8155 2777 50  0000 C CNN
-F 2 "" H 8150 2950 50  0001 C CNN
-F 3 "" H 8150 2950 50  0001 C CNN
-	1    8150 2950
-	1    0    0    -1
-$EndComp
-$Comp
-L power:GND #PWR0106
-U 1 1 5E88EDE8
-P 8550 2850
-F 0 "#PWR0106" H 8550 2600 50  0001 C CNN
-F 1 "GND" H 8555 2677 50  0000 C CNN
-F 2 "" H 8550 2850 50  0001 C CNN
-F 3 "" H 8550 2850 50  0001 C CNN
-	1    8550 2850
-	1    0    0    -1
-$EndComp
-Wire Wire Line
-	8550 2850 8550 2750
-Wire Wire Line
-	8550 2350 8550 2250
-Wire Wire Line
-	8250 2550 8150 2550
-Wire Wire Line
-	8150 2550 8150 2650
-Wire Wire Line
-	8150 2850 8150 2950
-Wire Wire Line
-	8150 2550 8050 2550
-Connection ~ 8150 2550
 Wire Wire Line
 	8700 5100 8700 5000
@@
 Wire Wire Line
 	3250 5100 3250 5000
-$Comp
-L Device:R_Small R6
-U 1 1 5E87C3A2
-P 8150 2750
-F 0 "R6" H 8209 2796 50  0000 L CNN
-F 1 "1k" H 8209 2705 50  0000 L CNN
-F 2 "Resistor_SMD:R_0603_1608Metric" H 8150 2750 50  0001 C CNN
-F 3 "~" H 8150 2750 50  0001 C CNN
-	1    8150 2750
-	1    0    0    -1
-$EndComp
 $Comp
 L Device:R_Small R5
@@
 A4
 Text GLabel 4100 2500 0    50   Input ~ 0
-D8
+D8_LED_POWER
 Text GLabel 4100 2800 0    50   Input ~ 0
 D3_LED
@@
 Text GLabel 4100 4200 0    50   Input ~ 0
 SCL
-Text GLabel 8050 2550 0    50   Input ~ 0
-D3_LED
 $Comp
 L power:GND #PWR0122
@@
 Text Notes 6700 4450 0    50   ~ 0
 12V if possible, otherwise 5V
-$Comp
-L power:GND #PWR0105
-U 1 1 5E89572E
-P 10100 2850
-F 0 "#PWR0105" H 10100 2600 50  0001 C CNN
-F 1 "GND" H 10105 2677 50  0000 C CNN
-F 2 "" H 10100 2850 50  0001 C CNN
-F 3 "" H 10100 2850 50  0001 C CNN
-	1    10100 2850
-	1    0    0    -1
-$EndComp
-Wire Wire Line
-	10100 2850 10100 2750
-Wire Wire Line
-	10100 2350 10100 2250
-Text GLabel 9600 2550 0    50   Input ~ 0
-D3_LED
-$Comp
-L Connector:Screw_Terminal_01x04 J2
-U 1 1 5E89857B
-P 8450 3900
-F 0 "J2" H 8530 3892 50  0000 L CNN
-F 1 "Screw_Terminal_01x04" H 8530 3801 50  0000 L CNN
-F 2 "TerminalBlock_Phoenix:TerminalBlock_Phoenix_MKDS-3-4-5.08_1x04_P5.08mm_Horizontal" H 8450 3900 50  0001 C CNN
-F 3 "~" H 8450 3900 50  0001 C CNN
-	1    8450 3900
-	1    0    0    -1
-$EndComp
 Wire Wire Line
 	8000 3900 8250 3900
-Wire Wire Line
-	8000 3800 8250 3800
 Text GLabel 8250 4000 0    50   Input ~ 0
-SWA
-Text GLabel 8250 4100 0    50   Input ~ 0
-SWB
-Text GLabel 8550 2250 0    50   Input ~ 0
-SWA
-Text GLabel 10100 2250 0    50   Input ~ 0
-SWB
-$Comp
-L Device:Q_NMOS_GSD Q2
-U 1 1 5E8A6696
-P 10000 2550
-F 0 "Q2" H 10206 2596 50  0000 L CNN
-F 1 "Q_NMOS_GSD" H 10206 2505 50  0000 L CNN
-F 2 "Package_TO_SOT_SMD:SOT-23" H 10200 2650 50  0001 C CNN
-F 3 "~" H 10000 2550 50  0001 C CNN
-	1    10000 2550
-	1    0    0    -1
-$EndComp
-$Comp
-L Device:Q_NMOS_GSD Q1
-U 1 1 5E8A804C
-P 8450 2550
-F 0 "Q1" H 8656 2596 50  0000 L CNN
-F 1 "Q_NMOS_GSD" H 8656 2505 50  0000 L CNN
-F 2 "Package_TO_SOT_SMD:SOT-23" H 8650 2650 50  0001 C CNN
-F 3 "~" H 8450 2550 50  0001 C CNN
-	1    8450 2550
-	1    0    0    -1
-$EndComp
-$Comp
-L power:+12V #PWR0130
-U 1 1 5E890108
-P 8500 1250
-F 0 "#PWR0130" H 8500 1100 50  0001 C CNN
-F 1 "+12V" H 8515 1423 50  0000 C CNN
-F 2 "" H 8500 1250 50  0001 C CNN
-F 3 "" H 8500 1250 50  0001 C CNN
-	1    8500 1250
-	1    0    0    -1
-$EndComp
-$Comp
-L Device:Q_PMOS_GDS Q3
-U 1 1 5E88F1EF
-P 8400 1500
-F 0 "Q3" H 8606 1454 50  0000 L CNN
-F 1 "Q_PMOS_GDS" H 8606 1545 50  0000 L CNN
-F 2 "" H 8600 1600 50  0001 C CNN
-F 3 "~" H 8400 1500 50  0001 C CNN
-	1    8400 1500
-	1    0    0    1
-$EndComp
-Wire Wire Line
-	8500 1250 8500 1300
-Wire Wire Line
-	8500 1700 8500 1750
-Text GLabel 8500 1750 0    50   Input ~ 0
-SWA
-$Comp
-L Device:Q_PMOS_GDS Q4
-U 1 1 5E89A113
-P 9850 1500
-F 0 "Q4" H 10056 1454 50  0000 L CNN
-F 1 "Q_PMOS_GDS" H 10056 1545 50  0000 L CNN
-F 2 "" H 10050 1600 50  0001 C CNN
-F 3 "~" H 9850 1500 50  0001 C CNN
-	1    9850 1500
-	1    0    0    1
-$EndComp
-Text GLabel 9950 1750 0    50   Input ~ 0
-SWB
-Wire Wire Line
-	9950 1700 9950 1750
-$Comp
-L power:+12V #PWR0131
-U 1 1 5E89CF4D
-P 9950 1250
-F 0 "#PWR0131" H 9950 1100 50  0001 C CNN
-F 1 "+12V" H 9965 1423 50  0000 C CNN
-F 2 "" H 9950 1250 50  0001 C CNN
-F 3 "" H 9950 1250 50  0001 C CNN
-	1    9950 1250
-	1    0    0    -1
-$EndComp
-Wire Wire Line
-	9950 1250 9950 1300
-Text GLabel 8150 1500 0    50   Input ~ 0
-D4_PMOS_SWA
-Text GLabel 9600 1500 0    50   Input ~ 0
-D9_PMOS_SWA
+LED
 Text GLabel 4100 2700 0    50   Input ~ 0
 D4_PMOS_SWA
@@
 D9_PMOS_SWA
 Wire Wire Line
-	9600 2550 9800 2550
-Wire Wire Line
 	3650 5000 4100 5000
 Wire Wire Line
 	3250 5000 3450 5000
+$Comp
+L Device:Fuse_Small F1
+U 1 1 5E8EDDED
+P 8150 3800
+F 0 "F1" H 8150 3985 50  0000 C CNN
+F 1 "Fuse_Small" H 8150 3894 50  0000 C CNN
+F 2 "Private Fuses:ATO_Fuseholder_3522-2" H 8150 3800 50  0001 C CNN
+F 3 "~" H 8150 3800 50  0001 C CNN
+	1    8150 3800
+	1    0    0    -1
+$EndComp
+Wire Wire Line
+	8050 3800 7850 3800
+$Comp
+L Device:Q_PMOS_GDS Q4
+U 1 1 5E8D9806
+P 8450 1400
+F 0 "Q4" H 8656 1354 50  0000 L CNN
+F 1 "Q_PMOS_GDS" H 8656 1445 50  0000 L CNN
+F 2 "Package_TO_SOT_SMD:TO-252-2" H 8650 1500 50  0001 C CNN
+F 3 "~" H 8450 1400 50  0001 C CNN
+	1    8450 1400
+	1    0    0    1
+$EndComp
+Text GLabel 7400 1600 0    50   Input ~ 0
+D8_LED_POWER
+$Comp
+L Device:R_Small R8
+U 1 1 5E8DD06B
+P 8100 1200
+F 0 "R8" H 8159 1246 50  0000 L CNN
+F 1 "1k" H 8159 1155 50  0000 L CNN
+F 2 "Resistor_SMD:R_0603_1608Metric" H 8100 1200 50  0001 C CNN
+F 3 "~" H 8100 1200 50  0001 C CNN
+	1    8100 1200
+	1    0    0    -1
+$EndComp
+Wire Wire Line
+	8100 1300 8100 1400
+Connection ~ 8100 1400
+Wire Wire Line
+	8100 1400 8250 1400
+Wire Wire Line
+	8100 1050 8100 1100
+$Comp
+L Device:Q_NMOS_GSD Q3
+U 1 1 5E8E26D6
+P 7750 1600
+F 0 "Q3" H 7956 1646 50  0000 L CNN
+F 1 "Q_NMOS_GSD" H 7956 1555 50  0000 L CNN
+F 2 "Package_TO_SOT_SMD:SOT-23" H 7950 1700 50  0001 C CNN
+F 3 "~" H 7750 1600 50  0001 C CNN
+	1    7750 1600
+	1    0    0    -1
+$EndComp
+$Comp
+L power:+12V #PWR0103
+U 1 1 5E8E3DBC
+P 8100 1050
+F 0 "#PWR0103" H 8100 900 50  0001 C CNN
+F 1 "+12V" H 8115 1223 50  0000 C CNN
+F 2 "" H 8100 1050 50  0001 C CNN
+F 3 "" H 8100 1050 50  0001 C CNN
+	1    8100 1050
+	1    0    0    -1
+$EndComp
+$Comp
+L power:GND #PWR0112
+U 1 1 5E8E4636
+P 7850 1850
+F 0 "#PWR0112" H 7850 1600 50  0001 C CNN
+F 1 "GND" H 7855 1677 50  0000 C CNN
+F 2 "" H 7850 1850 50  0001 C CNN
+F 3 "" H 7850 1850 50  0001 C CNN
+	1    7850 1850
+	1    0    0    -1
+$EndComp
+Wire Wire Line
+	7850 1850 7850 1800
+Wire Wire Line
+	7400 1600 7500 1600
+$Comp
+L Device:R_Small R7
+U 1 1 5E8E852C
+P 7500 1750
+F 0 "R7" H 7559 1796 50  0000 L CNN
+F 1 "1k" H 7559 1705 50  0000 L CNN
+F 2 "Resistor_SMD:R_0603_1608Metric" H 7500 1750 50  0001 C CNN
+F 3 "~" H 7500 1750 50  0001 C CNN
+	1    7500 1750
+	1    0    0    -1
+$EndComp
+$Comp
+L power:GND #PWR0130
+U 1 1 5E8E896B
+P 7500 1900
+F 0 "#PWR0130" H 7500 1650 50  0001 C CNN
+F 1 "GND" H 7505 1727 50  0000 C CNN
+F 2 "" H 7500 1900 50  0001 C CNN
+F 3 "" H 7500 1900 50  0001 C CNN
+	1    7500 1900
+	1    0    0    -1
+$EndComp
+Wire Wire Line
+	7500 1900 7500 1850
+Wire Wire Line
+	7500 1650 7500 1600
+Connection ~ 7500 1600
+Wire Wire Line
+	7500 1600 7550 1600
+$Comp
+L power:+12V #PWR0104
+U 1 1 5E8F910E
+P 8550 1050
+F 0 "#PWR0104" H 8550 900 50  0001 C CNN
+F 1 "+12V" H 8565 1223 50  0000 C CNN
+F 2 "" H 8550 1050 50  0001 C CNN
+F 3 "" H 8550 1050 50  0001 C CNN
+	1    8550 1050
+	1    0    0    -1
+$EndComp
+Wire Wire Line
+	8550 1050 8550 1200
+Text GLabel 8550 1750 2    50   Input ~ 0
+LED
+$Comp
+L Connector:Screw_Terminal_01x03 J2
+U 1 1 5E8FEA19
+P 8450 3900
+F 0 "J2" H 8530 3942 50  0000 L CNN
+F 1 "Screw_Terminal_01x03" H 8530 3851 50  0000 L CNN
+F 2 "TerminalBlock_Phoenix:TerminalBlock_Phoenix_MKDS-1,5-3_1x03_P5.00mm_Horizontal" H 8450 3900 50  0001 C CNN
+F 3 "~" H 8450 3900 50  0001 C CNN
+	1    8450 3900
+	1    0    0    -1
+$EndComp
+Wire Wire Line
+	8550 1600 8550 1750
+Wire Wire Line
+	7850 1400 8100 1400
 $EndSCHEMATC
