File: hardware/led-dimmer/led_dimmer.sch (KiCad schematic (older format))
At the start: 23 parts, among them J1 USB_B_Micro, J2 Screw_Terminal_01x03, Q3 Q_NMOS_GSD, Q4 Q_PMOS_GDS, SW1 Rotary_Encoder_Switch, U1 ATSAMD21G18A-AUT, U2 LD1117S33TR_SOT223

Commit message: Changed to a 4-terminal block
Parts:
- removed J2: Screw_Terminal_01x03, TerminalBlock_Phoenix:TerminalBlock_Phoenix_MKDS-1,5-3_1x03_P5.00mm_Horizontal, symbol Connector:Screw_Terminal_01x03
- added J2: Screw_Terminal_01x04, TerminalBlock_Phoenix:TerminalBlock_Phoenix_MKDS-1,5-4_1x04_P5.00mm_Horizontal, symbol Connector:Screw_Terminal_01x04
- added R6, R9: 1k, Resistor_SMD:R_0603_1608Metric, symbol Device:R_Small
- F1: value Fuse_Small -> 5A
Connections:
- net labels added: A1_BATVOLT
- net labels removed: A1
- wire segments 69 -> 75
Changed lines of the file:
@@
 ~RESET
 Text GLabel 6100 2100 2    50   Input ~ 0
-A1
+A1_BATVOLT
 Text GLabel 6100 2200 2    50   Input ~ 0
 A2
@@
 12V if possible, otherwise 5V
 Wire Wire Line
-	8000 3900 8250 3900
-Text GLabel 8250 4000 0    50   Input ~ 0
+	8000 3900 8150 3900
+Text GLabel 8250 4100 0    50   Input ~ 0
 LED
 Text GLabel 4100 2700 0    50   Input ~ 0
@@
 P 8150 3800
 F 0 "F1" H 8150 3985 50  0000 C CNN
-F 1 "Fuse_Small" H 8150 3894 50  0000 C CNN
+F 1 "5A" H 8150 3894 50  0000 C CNN
 F 2 "Private Fuses:ATO_Fuseholder_3522-2" H 8150 3800 50  0001 C CNN
 F 3 "~" H 8150 3800 50  0001 C CNN
@@
 Text GLabel 8550 1750 2    50   Input ~ 0
 LED
-$Comp
-L Connector:Screw_Terminal_01x03 J2
-U 1 1 5E8FEA19
+Wire Wire Line
+	8550 1600 8550 1750
+Wire Wire Line
+	7850 1400 8100 1400
+$Comp
+L Device:R_Small R6
+U 1 1 5E9692E7
+P 7500 3650
+F 0 "R6" H 7559 3696 50  0000 L CNN
+F 1 "1k" H 7559 3605 50  0000 L CNN
+F 2 "Resistor_SMD:R_0603_1608Metric" H 7500 3650 50  0001 C CNN
+F 3 "~" H 7500 3650 50  0001 C CNN
+	1    7500 3650
+	-1   0    0    1
+$EndComp
+$Comp
+L Device:R_Small R9
+U 1 1 5E96A36E
+P 7500 3950
+F 0 "R9" H 7559 3996 50  0000 L CNN
+F 1 "1k" H 7559 3905 50  0000 L CNN
+F 2 "Resistor_SMD:R_0603_1608Metric" H 7500 3950 50  0001 C CNN
+F 3 "~" H 7500 3950 50  0001 C CNN
+	1    7500 3950
+	-1   0    0    1
+$EndComp
+Wire Wire Line
+	7500 3750 7500 3800
+$Comp
+L power:GND #PWR0105
+U 1 1 5E97387E
+P 7500 4050
+F 0 "#PWR0105" H 7500 3800 50  0001 C CNN
+F 1 "GND" H 7505 3877 50  0000 C CNN
+F 2 "" H 7500 4050 50  0001 C CNN
+F 3 "" H 7500 4050 50  0001 C CNN
+	1    7500 4050
+	1    0    0    -1
+$EndComp
+$Comp
+L power:+12V #PWR0106
+U 1 1 5E973AB6
+P 7500 3550
+F 0 "#PWR0106" H 7500 3400 50  0001 C CNN
+F 1 "+12V" H 7515 3723 50  0000 C CNN
+F 2 "" H 7500 3550 50  0001 C CNN
+F 3 "" H 7500 3550 50  0001 C CNN
+	1    7500 3550
+	1    0    0    -1
+$EndComp
+Wire Wire Line
+	7500 3800 7350 3800
+Connection ~ 7500 3800
+Wire Wire Line
+	7500 3800 7500 3850
+Text GLabel 7350 3800 0    50   Input ~ 0
+A1_BATVOLT
+$Comp
+L Connector:Screw_Terminal_01x04 J2
+U 1 1 5E9E6490
 P 8450 3900
-F 0 "J2" H 8530 3942 50  0000 L CNN
-F 1 "Screw_Terminal_01x03" H 8530 3851 50  0000 L CNN
-F 2 "TerminalBlock_Phoenix:TerminalBlock_Phoenix_MKDS-1,5-3_1x03_P5.00mm_Horizontal" H 8450 3900 50  0001 C CNN
+F 0 "J2" H 8530 3892 50  0000 L CNN
+F 1 "Screw_Terminal_01x04" H 8530 3801 50  0000 L CNN
+F 2 "TerminalBlock_Phoenix:TerminalBlock_Phoenix_MKDS-1,5-4_1x04_P5.00mm_Horizontal" H 8450 3900 50  0001 C CNN
 F 3 "~" H 8450 3900 50  0001 C CNN
 	1    8450 3900
@@
 $EndComp
 Wire Wire Line
-	8550 1600 8550 1750
-Wire Wire Line
-	7850 1400 8100 1400
+	8250 4000 8150 4000
+Wire Wire Line
+	8150 4000 8150 3900
+Connection ~ 8150 3900
+Wire Wire Line
+	8150 3900 8250 3900
 $EndSCHEMATC

Commit message: Update led_dimmer.sch
Parts:
- added C? (x2): 6.8pF, Capacitor_SMD:C_0603_1608Metric, symbol Device:C_Small
- added Y?: 32.768kHz, symbol Device:Crystal_Small
- SWD1: symbol connector:SWD_TAGCONNECT -> led_dimmer-rescue:SWD_TAGCONNECT-connector
Connections:
- net labels added: XIN32, XOUT32
- wire segments 75 -> 81
