File: hardware/power-distribution-complete/power-distribution-complete.kicad_pcb (KiCad board)
At the start: 2 copper layers, 140 parts, among them J1 12V, J10 Parallell, J11 Parallell, J12 Parallell, J13 Parallell, J14 Parallell, J15 Parallell, J16 Parallell, J17 Parallell, J18 POUT, J19 POUT, J2 GND, J20 POUT, J21 POUT, J22 POUT, J23 POUT, J24 POUT, J25 POUT, J26 POUT, J27 POUT, J28 POUT, J29 POUT, J3 Parallell, J30 POUT, J31 POUT, J32 POUT, J33 POUT, J34 POUT, J35 POUT, J36 POUT, J37 POUT, J38 CTRL, J39 M6 Battery input, J4 Parallell, J40 M6 Battery input, J5 Parallell, J6 Parallell, J7 Parallell, J8 Parallell, J9 Parallell, Q1 Q_PMOS_GDS, Q10 Q_PMOS_GDS, Q11 Q_PMOS_GDS, Q12 Q_PMOS_GDS, Q13 Q_PMOS_GDS, Q14 Q_PMOS_GDS, Q15 Q_PMOS_GDS, Q16 Q_PMOS_GDS, Q17 Q_NMOS_SGD, Q18 Q_NMOS_SGD, Q19 Q_NMOS_SGD, Q2 Q_PMOS_GDS, Q20 Q_NMOS_SGD, Q21 Q_NMOS_SGD, Q22 Q_NMOS_SGD, Q3 Q_PMOS_GDS, Q4 Q_PMOS_GDS, Q5 Q_PMOS_GDS, Q6 Q_PMOS_GDS, Q7 Q_PMOS_GDS, Q8 Q_PMOS_GDS, Q9 Q_PMOS_GDS, U1 LTC4365TS8

Commit message: Updated the power distribution schematic and pcb
Parts:
- removed J1: 12V, Private:M5_7461383
- removed J10: Parallell, Connector_PinHeader_2.54mm:PinHeader_1x02_P2.54mm_Vertical
- removed J2: GND, Private:M5_7461383
- removed J38: CTRL, TerminalBlock_Phoenix:TerminalBlock_Phoenix_MKDS-1,5-6_1x06_P5.00mm_Horizontal
- added D1: D_Small, diode:SlimSMA_DO-221AC-2, F.Cu at (82.0, 94.0)
- added D17: D_Small, diode:SlimSMA_DO-221AC-2, F.Cu at (278.0, 94.0)
- added D18: D_Small, diode:SlimSMA_DO-221AC-2, F.Cu at (278.0, 114.0)
- added D19: D_Small, diode:SlimSMA_DO-221AC-2, F.Cu at (278.0, 134.0)
- added D2: D_Small, diode:SlimSMA_DO-221AC-2, F.Cu at (82.0, 114.0)
- added D20: D_Small, diode:SlimSMA_DO-221AC-2, F.Cu at (278.0, 154.0)
- added D21: D_Small, diode:SlimSMA_DO-221AC-2, F.Cu at (278.0, 174.0)
- added D22: D_Small, diode:SlimSMA_DO-221AC-2, F.Cu at (278.0, 194.0)
- added D23: D_Small, diode:SlimSMA_DO-221AC-2, F.Cu at (278.0, 214.0)
- added D24: D_Small, diode:SlimSMA_DO-221AC-2, F.Cu at (278.0, 234.0)
- added D3: D_Small, diode:SlimSMA_DO-221AC-2, F.Cu at (82.0, 134.0)
- added D4: D_Small, diode:SlimSMA_DO-221AC-2, F.Cu at (82.0, 154.0)
- added D5: D_Small, diode:SlimSMA_DO-221AC-2, F.Cu at (82.0, 174.0)
- added D6: D_Small, diode:SlimSMA_DO-221AC-2, F.Cu at (82.0, 194.0)
- added D7: D_Small, diode:SlimSMA_DO-221AC-2, F.Cu at (82.0, 214.0)
- added D8: D_Small, diode:SlimSMA_DO-221AC-2, F.Cu at (82.0, 234.0)
- added R1: 10k, Resistor_SMD:R_0603_1608Metric_Pad1.05x0.95mm_HandSolder, F.Cu at (137.0, 91.0)
- added R10: 10k, Resistor_SMD:R_0603_1608Metric_Pad1.05x0.95mm_HandSolder, F.Cu at (222.0, 201.0)
- added R11: 10k, Resistor_SMD:R_0603_1608Metric_Pad1.05x0.95mm_HandSolder, F.Cu at (222.0, 181.0)
- added R12: 10k, Resistor_SMD:R_0603_1608Metric_Pad1.05x0.95mm_HandSolder, F.Cu at (222.0, 161.0)
- added R13: 10k, Resistor_SMD:R_0603_1608Metric_Pad1.05x0.95mm_HandSolder, F.Cu at (222.0, 81.0)
- added R14: 10k, Resistor_SMD:R_0603_1608Metric_Pad1.05x0.95mm_HandSolder, F.Cu at (222.0, 101.0)
- added R15: 10k, Resistor_SMD:R_0603_1608Metric_Pad1.05x0.95mm_HandSolder, F.Cu at (222.0, 121.0)
- added R16: 10k, Resistor_SMD:R_0603_1608Metric_Pad1.05x0.95mm_HandSolder, F.Cu at (222.0, 141.0)
- added R2: 10k, Resistor_SMD:R_0603_1608Metric_Pad1.05x0.95mm_HandSolder, F.Cu at (137.0, 111.0)
- added R3: 10k, Resistor_SMD:R_0603_1608Metric_Pad1.05x0.95mm_HandSolder, F.Cu at (137.0, 131.0)
- added R4: 10k, Resistor_SMD:R_0603_1608Metric_Pad1.05x0.95mm_HandSolder, F.Cu at (137.0, 151.0)
- added R5: 10k, Resistor_SMD:R_0603_1608Metric_Pad1.05x0.95mm_HandSolder, F.Cu at (137.0, 231.0)
- added R6: 10k, Resistor_SMD:R_0603_1608Metric_Pad1.05x0.95mm_HandSolder, F.Cu at (137.0, 211.0)
- added R7: 10k, Resistor_SMD:R_0603_1608Metric_Pad1.05x0.95mm_HandSolder, F.Cu at (137.0, 191.0)
- added R8: 10k, Resistor_SMD:R_0603_1608Metric_Pad1.05x0.95mm_HandSolder, F.Cu at (137.0, 171.0)
- added R9: 10k, Resistor_SMD:R_0603_1608Metric_Pad1.05x0.95mm_HandSolder, F.Cu at (222.0, 221.0)
- added REF**: MountingHole_3.2mm_M3_Pad_Via, MountingHole:MountingHole_3.2mm_M3_Pad_Via, F.Cu at (165.0, 190.0)
- added REF**: MountingHole_3.2mm_M3_Pad_Via, MountingHole:MountingHole_3.2mm_M3_Pad_Via, F.Cu at (245.0, 75.0)
- added REF**: MountingHole_3.2mm_M3_Pad_Via, MountingHole:MountingHole_3.2mm_M3_Pad_Via, F.Cu at (245.0, 240.0)
- added REF**: MountingHole_3.2mm_M3_Pad_Via, MountingHole:MountingHole_3.2mm_M3_Pad_Via, F.Cu at (115.0, 240.0)
- added REF**: MountingHole_3.2mm_M3_Pad_Via, MountingHole:MountingHole_3.2mm_M3_Pad_Via, F.Cu at (165.0, 140.0)
- added REF**: MountingHole_3.2mm_M3_Pad_Via, MountingHole:MountingHole_3.2mm_M3_Pad_Via, F.Cu at (165.0, 90.0)
- added REF**: MountingHole_3.2mm_M3_Pad_Via, MountingHole:MountingHole_3.2mm_M3_Pad_Via, F.Cu at (275.0, 30.0)
- added REF**: MountingHole_3.2mm_M3_Pad_Via, MountingHole:MountingHole_3.2mm_M3_Pad_Via, F.Cu at (85.0, 30.0)
- added REF**: MountingHole_3.2mm_M3_Pad_Via, MountingHole:MountingHole_3.2mm_M3_Pad_Via, F.Cu at (195.0, 90.0)
- added REF**: MountingHole_3.2mm_M3_Pad_Via, MountingHole:MountingHole_3.2mm_M3_Pad_Via, F.Cu at (195.0, 140.0)
- added REF**: MountingHole_3.2mm_M3_Pad_Via, MountingHole:MountingHole_3.2mm_M3_Pad_Via, F.Cu at (195.0, 190.0)
- added REF**: MountingHole_3.2mm_M3_Pad_Via, MountingHole:MountingHole_3.2mm_M3_Pad_Via, F.Cu at (115.0, 75.0)
- added SWITCH_A5: ON/OFF, connectors:TerminalBlock_02_P5.00mm, F.Cu at (182.0, 30.0)
- G_PD1, Q17, Q18, Q20, R_LED_IN1, R_LED_OUT1, SHDN_PD1, U1, UV1, UV2, UV3: moved to B.Cu
- Q1, Q10, Q11, Q12, Q13, Q14, Q15, Q16, Q2, Q3, Q4, Q5, Q6, Q7, Q8, Q9: footprint Package_TO_SOT_SMD:TO-252-2 -> mosfet:TO-252-2-ThermalVias
- SWITCH_A1, SWITCH_A2, SWITCH_A3, SWITCH_A4, SWITCH_B1, SWITCH_B2, SWITCH_B3, SWITCH_B4, SWITCH_C1, SWITCH_C2, SWITCH_C3, SWITCH_C4, SWITCH_C5, SWITCH_C6, SWITCH_C7, SWITCH_C8: footprint TerminalBlock_Phoenix:TerminalBlock_Phoenix_PT-1,5-2-5.0-H_1x02_P5.00mm_Horizontal -> connectors:TerminalBlock_02_P5.00mm
- moved J11 436.3 mm to (265.5, 6.00), turned to 270 degrees
- moved SWITCH_A3 415.1 mm to (262.0, 30.0), turned to 180 degrees
- moved J13 414.5 mm to (245.5, 6.00), turned to 270 degrees
- moved J12 398.8 mm to (255.5, 6.00), turned to 270 degrees
- moved J4 394.6 mm to (145.5, 6.00), turned to 270 degrees
- moved J8 392.9 mm to (103.0, 6.00), turned to 90 degrees
- moved SWITCH_B3 388.4 mm to (252.0, 30.0), turned to 180 degrees
- moved Q1 387.9 mm to (134.1, 86.0), turned to 180 degrees
- moved SWITCH_C5 385.5 mm to (242.0, 30.0), turned to 180 degrees
- moved J14 383.5 mm to (235.5, 6.00), turned to 270 degrees
- moved F1 380.7 mm to (116.0, 86.0), turned to 0 degrees
- moved J33 379.6 mm to (274.0, 230.0), turned to 90 degrees
- moved SWITCH_C8 375.4 mm to (222.0, 30.0), turned to 180 degrees
- moved SWITCH_A1 373.7 mm to (172.0, 30.0), turned to 180 degrees
- moved J18 371.9 mm to (85.4, 82.4), turned to 270 degrees
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Connections:
- net Net-(F17-Pad1) renamed /Output/OUTNM1
- net Net-(F18-Pad1) renamed /Output/OUTNM2
- net Net-(F19-Pad1) renamed /Output/OUTNM3
- net Net-(F20-Pad1) renamed /Output/OUTNM4
Routing:
- net 12V_in: track 0.00 -> 397.3 mm, vias 0 -> 3
- net ~SHDN: track 0.00 -> 385.0 mm, vias 0 -> 2
- net Net-(J7-Pad1): track 0.00 -> 278.6 mm, vias 0 -> 1
- net Net-(J7-Pad2): track 0.00 -> 267.9 mm, vias 0 -> 1
- net Net-(J11-Pad1): track 0.00 -> 262.4 mm, vias 0 -> 1
- net Net-(J8-Pad2): track 0.00 -> 257.1 mm, vias 0 -> 1
- net Net-(J11-Pad2): track 0.00 -> 251.1 mm, vias 0 -> 1
- net Net-(J6-Pad2): track 0.00 -> 246.3 mm, vias 0 -> 1
- net Net-(J12-Pad2): track 0.00 -> 240.3 mm, vias 0 -> 1
- net Net-(J5-Pad2): track 0.00 -> 235.5 mm, vias 0 -> 1
- net Net-(J13-Pad2): track 0.00 -> 229.6 mm, vias 0 -> 1
- net Net-(J4-Pad2): track 0.00 -> 225.2 mm, vias 0 -> 1
- net Net-(J14-Pad2): track 0.00 -> 218.8 mm, vias 0 -> 1
- net Net-(J3-Pad2): track 0.00 -> 213.9 mm, vias 0 -> 1
- net Net-(J16-Pad2): track 0.00 -> 208.0 mm, vias 0 -> 1
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- added copper zone on B.Cu, net +12V
- added copper zone on F.Cu, net +12V
- added copper zone on B.Cu, net /Output/AOUT
- added copper zone on F.Cu, net /Output/AOUT
- added copper zone on B.Cu, net /Output/BOUT
- added copper zone on F.Cu, net /Output/BOUT
- added copper zone on B.Cu, net /Output/COUT
- added copper zone on F.Cu, net /Output/COUT
- added copper zone on B.Cu, net /Output/DOUT
- added copper zone on F.Cu, net /Output/DOUT
- added copper zone on B.Cu, net /Output/EOUT
- added copper zone on F.Cu, net /Output/EOUT
- added copper zone on B.Cu, net /Output/FOUT
- added copper zone on F.Cu, net /Output/FOUT
- added copper zone on B.Cu, net /Output/GOUT
- added copper zone on F.Cu, net /Output/GOUT
- added copper zone on B.Cu, net /Output/HOUT
- added copper zone on F.Cu, net /Output/HOUT
- added copper zone on B.Cu, net /Output/IOUT
- added copper zone on F.Cu, net /Output/IOUT
- added copper zone on B.Cu, net /Output/JOUT
- added copper zone on F.Cu, net /Output/JOUT
- added copper zone on B.Cu, net /Output/KOUT
- added copper zone on F.Cu, net /Output/KOUT
- added copper zone on B.Cu, net /Output/LOUT
- added copper zone on F.Cu, net /Output/LOUT
- added copper zone on B.Cu, net /Output/MOUT
- added copper zone on F.Cu, net /Output/MOUT
- added copper zone on B.Cu, net /Output/NOUT
- added copper zone on F.Cu, net /Output/NOUT
- added copper zone on B.Cu, net /Output/OOUT
- added copper zone on F.Cu, net /Output/OOUT
- added copper zone on B.Cu, net /Output/OUTNM1
- added copper zone on F.Cu, net /Output/OUTNM1
- added copper zone on B.Cu, net /Output/OUTNM2
- added copper zone on F.Cu, net /Output/OUTNM2
- added copper zone on B.Cu, net /Output/OUTNM3
- added copper zone on F.Cu, net /Output/OUTNM3
- added copper zone on B.Cu, net /Output/OUTNM4
- added copper zone on F.Cu, net /Output/OUTNM4
- added copper zone on B.Cu, net /Output/POUT
- added copper zone on F.Cu, net /Output/POUT
- added copper zone on B.Cu, net 12V_in
- added copper zone on F.Cu, net 12V_in
- added copper zone on B.Cu, net GND
- added copper zone on F.Cu, net GND
- added copper zone on B.Cu, net SSR-A
- added copper zone on F.Cu, net SSR-A
- added copper zone on B.Cu, net SSR-B
- added copper zone on F.Cu, net SSR-B
- added copper zone on B.Cu, net SSR-C
- added copper zone on F.Cu, net SSR-C
- added copper zone on B.Cu, net SSR-D
- added copper zone on F.Cu, net SSR-D
- added copper zone on B.Cu, net SSR-E
- added copper zone on F.Cu, net SSR-E
- added copper zone on B.Cu, net SSR-F
- added copper zone on F.Cu, net SSR-F
- added copper zone on B.Cu, net SSR-G
- added copper zone on F.Cu, net SSR-G
- added copper zone on B.Cu, net SSR-H
- added copper zone on F.Cu, net SSR-H
- added copper zone on B.Cu, net SSR-I
- added copper zone on F.Cu, net SSR-I
- added copper zone on B.Cu, net SSR-J
- added copper zone on F.Cu, net SSR-J
- added copper zone on B.Cu, net SSR-K
- added copper zone on F.Cu, net SSR-K
- added copper zone on B.Cu, net SSR-L
- added copper zone on F.Cu, net SSR-L
- added copper zone on B.Cu, net SSR-M
- added copper zone on F.Cu, net SSR-M
- added copper zone on B.Cu, net SSR-N
- added copper zone on F.Cu, net SSR-N
- added copper zone on B.Cu, net SSR-O
- added copper zone on F.Cu, net SSR-O
- added copper zone on B.Cu, net SSR-P
- added copper zone on F.Cu, net SSR-P
Other:
- board outline added: 230 x 235 mm
- board text added: "1"
- board text added: "12 V"
- board text added: "12 V IN"
- board text added: "12 V OUT"
- board text added: "2"
- board text added: "3"
- board text added: "4"
- board text added: "A"
- board text added: "A |"
- board text added: "B"
- board text added: "B |"
- board text added: "BAT|"
- board text added: "C"
- board text added: "C |"
- board text added: "D"
- board text added: "D |"
- board text added: "E"
- board text added: "E |"
- board text added: "F"
- board text added: "F |"
- board text added: "G"
- board text added: "G |"
- board text added: "GND"
- board text added: "GND | SIG"
- board text added: "H"
- board text added: "I"
- board text added: "I |"
- board text added: "J"
- board text added: "J |"
- board text added: "K"
- board text added: "K |"
- board text added: "L"
- board text added: "L |"
- board text added: "M"
- board text added: "M |"
- board text added: "N"
- board text added: "N |"
- board text added: "O"
- board text added: "O |"
- board text added: "P"
- board text added: "P |"
- board text added: "SIG | 12V"
- board text added: "| H |"

Commit message: Power distribution complete first order
The board is finished and ordered.

Added TVS diode to protect the board from transients.
Parts:
- removed G_PD1: 10k, Resistor_SMD:R_0603_1608Metric
- added D33: D_Small, diode:SMF-DO-219AB, F.Cu at (278.1, 54.0)
- added D34: D_Small, diode:SMF-DO-219AB, F.Cu at (278.1, 74.0)
- added D35: D_Small, diode:SMF-DO-219AB, F.Cu at (82.0, 74.0)
- added D36: D_Small, diode:SMF-DO-219AB, F.Cu at (81.9, 54.0)
- added D37: D_Small, diode:SMF-DO-219AB, F.Cu at (198.5, 244.0)
- added D38: D_Small, diode:SMF-DO-219AB, F.Cu at (198.5, 248.0)
- added D39: D_Small, diode:SMF-DO-219AB, F.Cu at (198.5, 246.0)
- D1, D17, D18, D19, D2, D20, D21, D22, D23, D24, D3, D4, D5, D6, D7, D8: footprint diode:SlimSMA_DO-221AC-2 -> diode:SMF-DO-219AB
- R17, R18, R19, R20, R21, R22, R23, R24, R25, R26, R27, R28, R29, R30, R31, R32: value 670R -> 1k
- moved J7 213.6 mm to (129.0, 216.5)
- moved J11 213.0 mm to (230.0, 216.0)
- moved J8 191.8 mm to (129.0, 196.0)
- moved J12 191.7 mm to (230.0, 196.0)
- moved J9 170.8 mm to (129.0, 176.0)
- moved J13 170.7 mm to (230.0, 176.0)
- moved J14 150.1 mm to (230.0, 156.0)
- moved J6 150.0 mm to (129.0, 156.0), turned to 90 degrees
- moved J17 130.2 mm to (230.0, 136.0), turned to 270 degrees
- moved J5 130.2 mm to (129.0, 136.0), turned to 90 degrees
- moved J16 111.3 mm to (230.0, 116.0), turned to 270 degrees
- moved J4 111.2 mm to (129.0, 116.0), turned to 90 degrees
- moved J15 94.0 mm to (230.0, 96.0), turned to 270 degrees
- moved J3 93.8 mm to (129.0, 96.0), turned to 90 degrees
Routing:
- net Net-(J11-Pad2): track 251.1 -> 325.3 mm
- net Net-(J12-Pad2): track 240.3 -> 313.8 mm
- net Net-(J13-Pad2): track 229.6 -> 302.6 mm
- net Net-(J14-Pad2): track 218.8 -> 290.1 mm
- net Net-(J16-Pad2): track 208.0 -> 276.5 mm
- net Net-(J15-Pad2): track 197.2 -> 265.0 mm
- net Net-(J15-Pad1): track 186.1 -> 249.5 mm
- net Net-(J5-Pad2): track 235.5 -> 291.7 mm
- net Net-(J4-Pad2): track 225.2 -> 280.8 mm
- net Net-(J6-Pad2): track 246.3 -> 301.8 mm
- net Net-(J3-Pad2): track 213.9 -> 268.8 mm
- net Net-(J7-Pad2): track 267.9 -> 321.8 mm
- net Net-(J8-Pad2): track 257.1 -> 309.8 mm
- net Net-(J7-Pad1): track 278.6 -> 328.8 mm
- net 12V_in: track 397.3 -> 432.2 mm
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Other:
- board text added: "Power distribution board Max 15 A fuse."
- board text added: "Rev 5 - 2021-01"
- board text added: "The board has a under-voltage protection and turns off if the battery voltage becomes to low. The |sig|12V| terminal should be shorted to turn on the battery. The |gnd|sig| terminal should be shorted to turn on the corresponding output."
- board text added: "UV Protection set by UV2 12.00 V - 434 Ohm 11.75 V - 444 Ohm 11.50 V - 454 Ohm 11.25 V - 465 Ohm"
